Commit message: Update robot.xacro

File: robot_description_pkg/urdf/robot.xacro (robot description, xacro)
@@ -169,15 +169,12 @@
             <origin xyz="0.0 0.0 0.0" rpy="0.0 0.0 0.0"/>
             <geometry>
-                <mesh filename="package://robot_description_pkg/meshes/hokuyo_2.dae"/>
+                <mesh filename="package://robot_description_pkg/meshes/hokuyo.dae"/>
             </geometry>
-            <material name="">
-                <color rgba="1.0 0.0 0.0 1.0"/>
-                <texture filename=""/>
-            </material>
+            <material name="Red">
         </visual>
         <collision>
             <origin xyz="0.0 0.0 0.0" rpy="0.0 0.0 0.0"/>
             <geometry>
-                <box size="0.0 0.0 0.0"/>
+                <mesh filename="package://robot_description_pkg/meshes/hokuyo.dae"/>
             </geometry>
         </collision>

Commit message: Update robot.xacro

File: robot_description_pkg/urdf/robot.xacro (robot description, xacro)
@@ -160,5 +160,5 @@
     </joint>
     <!-- LIDAR LINK -->
-    <link name="link_name">
+    <link name="lider">
         <inertial>
             <origin xyz="0.0 0.0 0.0" rpy="0.0 0.0 0.0"/>
@@ -180,5 +180,4 @@
         </collision>
     </link>
-<!--
     <joint name="lider_joint" type="fixed">
         <origin xyz="0 0 0.304" rpy="0 0 0"/>
@@ -187,4 +186,3 @@
         <axis xyz="0 0 0" />
     </joint>
--->
 </robot>

Commit message: Update robot.xacro

File: robot_description_pkg/urdf/robot.xacro (robot description, xacro)
@@ -24,6 +24,6 @@
         </collision>
     </link>
-    <!-- FRIST RIGHT WHEEL LINK -->
-    <link name="frist_right_wheel">
+    <!-- FRONT RIGHT WHEEL LINK -->
+    <link name="front_right_wheel">
         <inertial>
             <origin xyz="0.0 0.0 0.0" rpy="0.0 0.0 0.0"/>
@@ -45,12 +45,12 @@
         </collision>
     </link>
-    <joint name="frist_right_wheel_joint" type="continuous">
+    <joint name="front_right_wheel_joint" type="continuous">
         <origin xyz="0.175 0.24 0.10" rpy="0.0 0.0 0.0"/>
         <parent link="chassis"/>
-        <child link="frist_right_wheel"/>
+        <child link="front_right_wheel"/>
         <axis xyz="0 0 0"/>
     </joint>
-    <!-- SECOND RIGHT WHEEL LINK -->
-    <link name="second_right_wheel">
+    <!-- BACk RIGHT WHEEL LINK -->
+    <link name="back_right_wheel">
         <inertial>
             <origin rpy="0.0 0.0 0.0"/>
@@ -72,12 +72,12 @@
         </collision>
     </link>
-    <joint name="second_right_wheel_joint" type="continuous">
+    <joint name="back_right_wheel_joint" type="continuous">
         <origin xyz="-0.175 0.24 0.10" rpy="0.0 0.0 0.0"/>
         <parent link="chassis"/>
-        <child link="second_right_wheel"/>
+        <child link="back_right_wheel"/>
         <axis xyz="0 0 0"/>
     </joint>
-    <!-- FRIST LEFT WHEEL LINK -->
-    <link name="frist_left_wheel">
+    <!-- FRONT LEFT WHEEL LINK -->
+    <link name="front_left_wheel">
         <inertial>
             <origin xyz="0.0 0.0 0.0" rpy="0.0 0.0 0.0"/>
@@ -99,12 +99,12 @@
         </collision>
     </link>
-    <joint name="frist_left_wheel_joint" type="continuous">
+    <joint name="front_left_wheel_joint" type="continuous">
         <origin xyz="0.175 -0.24 0.10" rpy="0.0 0.0 0.0"/>
         <parent link="chassis"/>
-        <child link="frist_left_wheel"/>
+        <child link="front_left_wheel"/>
         <axis xyz="0 0 0"/>
     </joint>
-    <!-- SECOND LEFT WHEEL LINK -->
-    <link name="second_left_wheel">
+    <!-- BACK LEFT WHEEL LINK -->
+    <link name="back_left_wheel">
         <inertial>
             <origin xyz="0.0 0.0 0.0" rpy="0.0 0.0 0.0"/>
@@ -126,8 +126,8 @@
         </collision>
     </link>
-    <joint name="second_left_wheel_joint" type="continuous">
+    <joint name="back_left_wheel_joint" type="continuous">
         <origin xyz="-0.175 -0.24 0.10" rpy="0.0 0.0 0.0"/>
         <parent link="chassis"/>
-        <child link="second_left_wheel"/>
+        <child link="back_left_wheel"/>
         <axis xyz="0 0 0"/>
     </joint>

Commit message: Update robot.xacro

File: robot_description_pkg/urdf/robot.xacro (robot description, xacro)
@@ -3,4 +3,6 @@
     <xacro:include filename="$(find robot_description_pkg)/urdf/material.xacro"/>
     <xacro:include filename="$(find robot_description_pkg)/urdf/gazebo.xacro"/>
+    <link name="base_link">
+    </link>
     <!-- CHASSIS LINK -->
     <link name="chassis">
@@ -24,4 +26,8 @@
         </collision>
     </link>
+    <joint name="joint_name" type="fixed">
+        <parent link="base_link"/>
+        <child link="chassis"/>
+    </joint>
     <!-- FRONT RIGHT WHEEL LINK -->
     <link name="front_right_wheel">

Commit message: Update robot.xacro

File: robot_description_pkg/urdf/robot.xacro (robot description, xacro)
@@ -1,13 +1,13 @@
 <?xml version="1.0"?>
-<robot xmlns:xacro="http://www.ros.org/wiki/xacro" name="my_robot">
-    <xacro:include filename="$(find robot_description_pkg)/urdf/material.xacro"/>
-    <xacro:include filename="$(find robot_description_pkg)/urdf/gazebo.xacro"/>
-    <link name="base_link">
-    </link>
-    <!-- CHASSIS LINK -->
-    <link name="chassis">
-        <inertial>s
+<robot xmlns:xacro="http://www.ros.org/wiki/xacro" name="myrobot">
+  <xacro:include filename="$(find robot_description_pkg)/urdf/material.xacro"/>
+  <xacro:include filename="$(find robot_description_pkg)/urdf/gazebo.xacro" />
+  <link name="base_link">
+  </link>
+  <!-- CHASSIS LINK -->
+  <link name="chassis">
+        <inertial>
             <origin xyz="0.0 0.0 0.0"/>
-            <mass value="1.0"/>
+            <mass value="0.30"/>
             <inertia ixx="0.1" ixy="0.0" ixz="0.0" iyy="0.1" iyz="0.0" izz="0.1"/>
         </inertial>
@@ -25,126 +25,126 @@
             </geometry>
         </collision>
-    </link>
-    <joint name="joint_name" type="fixed">
+  </link>
+  <joint name="joint_name" type="fixed">
         <parent link="base_link"/>
         <child link="chassis"/>
-    </joint>
-    <!-- FRONT RIGHT WHEEL LINK -->
-    <link name="front_right_wheel">
-        <inertial>
-            <origin xyz="0.0 0.0 0.0" rpy="0.0 0.0 0.0"/>
-            <mass value="0.0"/>
-            <inertia ixx="0.0" ixy="0.0" ixz="0.0" iyy="0.0" iyz="0.0" izz="0.0"/>
-        </inertial>
-        <visual >
-            <origin  rpy="0 1.5707 1.5707"/>
-            <geometry>
-                <cylinder radius="0.1" length="0.03"/>
-            </geometry>
-            <material name="Black"/>
-        </visual>
-        <collision>
-            <origin xrpy="0 1.5707 1.5707"/>
-            <geometry>
-                <cylinder radius=".1" length="0.03"/>
-            </geometry>
-        </collision>
-    </link>
-    <joint name="front_right_wheel_joint" type="continuous">
-        <origin xyz="0.175 0.24 0.10" rpy="0.0 0.0 0.0"/>
-        <parent link="chassis"/>
-        <child link="front_right_wheel"/>
-        <axis xyz="0 0 0"/>
-    </joint>
-    <!-- BACk RIGHT WHEEL LINK -->
-    <link name="back_right_wheel">
-        <inertial>
-            <origin rpy="0.0 0.0 0.0"/>
-            <mass value="0.0"/>
-            <inertia ixx="0.0" ixy="0.0" ixz="0.0" iyy="0.0" iyz="0.0" izz="0.0"/>
-        </inertial>
-        <visual >
-            <origin  rpy="0 1.5707 1.5707"/>
-            <geometry>
-                <cylinder radius="0.1" length="0.03"/>
-            </geometry>
-            <material name="Black"/>
-        </visual>
-        <collision>
-            <origin  rpy="0 1.5707 1.5707"/>
-            <geometry>
-                <cylinder radius=".1" length="0.03"/>
-            </geometry>
-        </collision>
-    </link>
-    <joint name="back_right_wheel_joint" type="continuous">
-        <origin xyz="-0.175 0.24 0.10" rpy="0.0 0.0 0.0"/>
-        <parent link="chassis"/>
-        <child link="back_right_wheel"/>
-        <axis xyz="0 0 0"/>
-    </joint>
-    <!-- FRONT LEFT WHEEL LINK -->
-    <link name="front_left_wheel">
-        <inertial>
-            <origin xyz="0.0 0.0 0.0" rpy="0.0 0.0 0.0"/>
-            <mass value="0.0"/>
-            <inertia ixx="0.0" ixy="0.0" ixz="0.0" iyy="0.0" iyz="0.0" izz="0.0"/>
-        </inertial>
-        <visual >
-            <origin  rpy="0 1.5707 1.5707"/>
-            <geometry>
-                <cylinder radius="0.1" length="0.03"/>
-            </geometry>
-            <material name="Black"/>
-        </visual>
-        <collision>
-            <origin rpy="0 1.5707 1.5707"/>
-            <geometry>
-                <cylinder radius=".1" length="0.03"/>
-            </geometry>
-        </collision>
-    </link>
-    <joint name="front_left_wheel_joint" type="continuous">
-        <origin xyz="0.175 -0.24 0.10" rpy="0.0 0.0 0.0"/>
-        <parent link="chassis"/>
-        <child link="front_left_wheel"/>
-        <axis xyz="0 0 0"/>
-    </joint>
-    <!-- BACK LEFT WHEEL LINK -->
-    <link name="back_left_wheel">
-        <inertial>
-            <origin xyz="0.0 0.0 0.0" rpy="0.0 0.0 0.0"/>
-            <mass value="0.0"/>
-            <inertia ixx="0.0" ixy="0.0" ixz="0.0" iyy="0.0" iyz="0.0" izz="0.0"/>
-        </inertial>
-        <visual >
-            <origin rpy="0 1.5707 1.5707"/>
-            <geometry>
-                <cylinder radius="0.1" length="0.03"/>
-            </geometry>
-            <material name="Black"/>
-        </visual>
-        <collision>
-            <origin rpy="0 1.5707 1.5707"/>
-            <geometry>
-                <cylinder radius=".1" length="0.03"/>
-            </geometry>
-        </collision>
-    </link>
-    <joint name="back_left_wheel_joint" type="continuous">
-        <origin xyz="-0.175 -0.24 0.10" rpy="0.0 0.0 0.0"/>
-        <parent link="chassis"/>
-        <child link="back_left_wheel"/>
-        <axis xyz="0 0 0"/>
-    </joint>
+  </joint>
+  <!-- FRONT RIGHT WHEEL LINK   -->
+  <link name="front_right_wheel">
+    <inertial>
+      <origin rpy="0 0 0 " xyz="0 0 0"/>
+      <mass value="0.2"/>
+      <inertia ixx="0.1" ixy="0" ixz="0" iyy="0.1" iyz="0" izz="0.1"/>
+    </inertial>
+    <collision name="front_right_wheel_collision">
+      <origin rpy="0 1.5707 1.5707" xyz="0 0 0" />
+      <geometry>
+        <cylinder length="0.04" radius="0.1"/>
+      </geometry>
+    </collision>
+    <visual name="front_right_wheel_visual">
+      <origin rpy="0 1.5707 1.5707" xyz="0 0 0"/>
+      <geometry>
+        <cylinder length="0.05" radius="0.1"/>
+      </geometry>
+      <material name="Black"/>
+    </visual>
+  </link>
+  <joint name="joint_front_right_wheel" type="continuous">
+    <origin rpy="0 0 0" xyz="0.175 0.25 0.1"/>
+    <child link="front_right_wheel" />
+    <parent link="chassis"/>
+    <axis rpy="0 0 0" xyz="0 1 0"/>
+  </joint>
+  <!-- BACk RIGHT WHEEL LINK    -->
+  <link name="back_right_wheel">
+    <inertial>
+      <mass value="0.2"/>
+      <origin rpy="0 0 0" xyz="0 0 0"/>
+      <inertia ixx="0.1" ixy="0" ixz="0" iyy="0.1" iyz="0" izz="0.1"/>
+    </inertial>
+    <collision name="back_right_wheel_collision">
+      <origin rpy="0 1.5707 1.5707" xyz="0 0 0" />
+      <geometry>
+        <cylinder length="0.04" radius="0.1"/>
+      </geometry>
+    </collision>
+    <visual name="back_right_wheel_visual">
+      <origin rpy="0 1.5707 1.5707" xyz="0 0 0"/>
+      <geometry>
+        <cylinder length="0.05" radius="0.1"/>
+      </geometry>
+      <material name="Black"/>
+    </visual>
+  </link>
+  <joint name="joint_back_right_wheel" type="continuous">
+    <origin rpy="0 0 0" xyz="-0.175 0.25 0.1"/>
+    <child link="back_right_wheel" />
+    <parent link="chassis"/>
+    <axis rpy="0 0 0" xyz="0 1 0"/>
+  </joint>
+  <!-- FRONT LEFTT WHEEL LINK   -->
+  <link name="front_left_wheel">
+    <inertial>
+      <mass value="0.2"/>
+      <origin rpy="0 0 0" xyz="0 0 0"/>
+      <inertia ixx="0.1" ixy="0" ixz="0" iyy="0.1" iyz="0" izz="0.1"/>
+    </inertial>
+    <collision name="front_left_wheel_collision">
+      <origin rpy="0 1.5707 1.5707" xyz="0 0 0" />
+      <geometry>
+        <cylinder length="0.05" radius="0.1"/>
+      </geometry>
+    </collision>
+    <visual name="front_left_wheel_visual">
+      <origin rpy="0 1.5707 1.5707" xyz="0 0 0"/>
+      <geometry>
+        <cylinder length="0.05" radius="0.1"/>
+      </geometry>
+      <material name="Black"/>
+    </visual>
+  </link>
+  <joint name="joint_front_left_wheel" type="continuous">
+    <origin rpy="0 0 0" xyz="0.175 -0.25 0.10"/>
+    <child link="front_left_wheel" />
+    <parent link="chassis"/>
+    <axis rpy="0 0 0" xyz="0 1 0"/>
+  </joint>
+<!-- BACk RIGHT WHEEL LINK    -->
+  <link name="back_left_wheel">
+    <inertial>
+      <mass value="0.2"/>
+      <origin rpy="0 0 0" xyz="0 0 0"/>
+      <inertia ixx="0.1" ixy="0" ixz="0" iyy="0.1" iyz="0" izz="0.1"/>
+    </inertial>
+    <collision name="back_left_wheel_collision">
+      <origin rpy="0 1.5707 1.5707" xyz="0 0 0" />
+      <geometry>
+        <cylinder length="0.04" radius="0.1"/>
+      </geometry>
+    </collision>
+    <visual name="back_left_wheel_visual">
+      <origin rpy="0 1.5707 1.5707" xyz="0 0 0"/>
+      <geometry>
+        <cylinder length="0.05" radius="0.1"/>
+      </geometry>
+      <material name="Black"/>
+    </visual>
+  </link>
+  <joint name="joint_back_left_wheel" type="continuous">
+    <origin rpy="0 0 0" xyz="-0.175 -0.25 0.10"/>
+    <child link="back_left_wheel" />
+    <parent link="chassis"/>
+    <axis rpy="0 0 0" xyz="0 1 0"/>
+  </joint>
     <!-- CAMERA LINK -->
     <link name="camera">
         <inertial>
             <origin xyz="0.0 0.0 0.0" rpy="0.0 0.0 0.0"/>
-            <mass value="0.0"/>
-            <inertia ixx="0.0" ixy="0.0" ixz="0.0" iyy="0.0" iyz="0.0" izz="0.0"/>
+            <mass value="0.01"/>
+            <inertia ixx="0.1" ixy="0.0" ixz="0.0" iyy="0.1" iyz="0.0" izz="0.1"/>
         </inertial>
         <visual >
-            <origin xyz="0.0 0.0 0.0" rpy="0.0 0.0 0.0"/>
+            <origin xyz="0.325 0.0 0.2" rpy="0 0 0"/>
             <geometry>
                 <box size="0.050 0.20 0.07"/>
@@ -153,12 +153,12 @@
         </visual>
         <collision>
-            <origin xyz="0.0 0.0 0.0" rpy="0.0 0.0 0.0"/>
+           <origin xyz="0.325 0.0 0.2" rpy="0 0 0"/>
             <geometry>
-                <box size="0.0 0.0 0.0"/>
+                <box size="0.050 0.20 0.07"/>
             </geometry>
         </collision>
     </link>
     <joint name="camera_link_joint" type="fixed">
-        <origin xyz="0.325 0.0 0.2" rpy="0.0 0.0 0.0"/>
+        <origin xyz="0 0 0" rpy="0.0 0.0 0.0"/>
         <parent link="chassis"/>
         <child link="camera"/>
@@ -167,25 +167,24 @@
     <!-- LIDAR LINK -->
     <link name="lider">
-        <inertial>
-            <origin xyz="0.0 0.0 0.0" rpy="0.0 0.0 0.0"/>
-            <mass value="0.0"/>
-            <inertia ixx="0.0" ixy="0.0" ixz="0.0" iyy="0.0" iyz="0.0" izz="0.0"/>
-        </inertial>
-        <visual name="">
-            <origin xyz="0.0 0.0 0.0" rpy="0.0 0.0 0.0"/>
-            <geometry>
-                <mesh filename="package://robot_description_pkg/meshes/hokuyo.dae"/>
-            </geometry>
-            <material name="Red">
-        </visual>
-        <collision>
-            <origin xyz="0.0 0.0 0.0" rpy="0.0 0.0 0.0"/>
-            <geometry>
-                <mesh filename="package://robot_description_pkg/meshes/hokuyo.dae"/>
-            </geometry>
-        </collision>
+    <inertial>
+        <origin xyz="0.0 0.0 0.0" rpy="0.0 0.0 0.0"/>
+        <mass value="0.10"/>
+        <inertia ixx="1.0" ixy="0.0" ixz="0.0" iyy="1.0" iyz="0.0" izz="1.0"/>
+    </inertial>
+    <visual>
+        <origin xyz=" 0 0 0" rpy="0 0 0"/>
+        <geometry>
+            <mesh filename="package://robot_description_pkg/meshes/hokuyo.dae"/>
+        </geometry>
+    </visual>
+    <collision>
+        <origin xyz="0.0 0.0 0.0" rpy="0.0 0.0 0.0"/>
+        <geometry>
+            <mesh filename="package://robot_description_pkg/meshes/hokuyo.dae" />
+        </geometry>
+    </collision>
     </link>
     <joint name="lider_joint" type="fixed">
-        <origin xyz="0 0 0.304" rpy="0 0 0"/>
+        <origin xyz="0.0 0.0 0.304" rpy="0 0 0"/>
         <parent link="chassis"/>
         <child link="lider"/>

Commit message: Update robot.xacro

File: robot_description_pkg/urdf/robot.xacro (robot description, xacro)
@@ -3,6 +3,12 @@
   <xacro:include filename="$(find robot_description_pkg)/urdf/material.xacro"/>
   <xacro:include filename="$(find robot_description_pkg)/urdf/gazebo.xacro" />
+ <link name="odom">
+  </link>
   <link name="base_link">
   </link>
+   <joint name="joint_base" type="fixed">
+        <parent link="odom"/>
+        <child link="base_link"/>
+  </joint>
   <!-- CHASSIS LINK -->
   <link name="chassis">
